File: pcb/ch549Board/simpleCH549_typeC.brd (EAGLE design)
At the start: 35.6 x 12 mm, 14 parts, among them J4 USB_A_SMT_MALE, U2 CH552G

Commit message: update pins in text editor
Parts:
- LED2: value P3.3 -> P2.2
- U2: value CH552G -> CH549G
Connections:
- net P3.3 renamed P2.2
- removed net P3.2: J2.5, U2.1
- new net P2.4: J2.7, U2.11
- net P1.1: now also J2.5, U2.1; no longer J1.2, U2.9
- net P3.0: now also J2.4, U2.7; no longer J2.3, U2.8
- net P3.1: now also J2.3, U2.8; no longer J2.4, U2.7
- net P3.4: now also J1.2, U2.9; no longer J2.7, U2.11
Routing:
- net P3.2: track 21.5 -> 0.00 mm, vias 3 -> 0
- net P2.4: track 0.00 -> 9.48 mm
- net P3.4: track 9.48 -> 17.2 mm, vias 0 -> 1
- net P1.1: track 17.2 -> 21.5 mm, vias 1 -> 3
- net P3.1: track 17.0 -> 17.5 mm
- net P3.0: track 17.5 -> 17.0 mm
Other:
- board text added: "P2.2"
- board text added: "P2.2 INT1"
- board text removed: "P3.3"
- board text removed: "P3.3 INT1"
Changed lines of the file:
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@@
 VBUS1
 AIN3</text>
-<text x="21.6408" y="10.0076" size="0.6096" layer="26" distance="30" rot="MR0" align="top-left">P3.3
+<text x="21.6408" y="10.0076" size="0.6096" layer="26" distance="30" rot="MR0" align="top-left">P2.2
 INT1</text>
 <text x="24.4348" y="10.0076" size="0.6096" layer="26" distance="30" rot="MR0" align="top-left">P3.4
@@
 <text x="6.7818" y="8.3312" size="0.8128" layer="26" distance="30" rot="MR0">Deqing Sun
 2023</text>
-<text x="25.654" y="2.3368" size="0.6096" layer="25">P3.3</text>
+<text x="25.654" y="2.3368" size="0.6096" layer="25">P2.2</text>
 <text x="25.654" y="9.0424" size="0.6096" layer="25">PWR</text>
 <text x="25.9588" y="4.4704" size="0.6096" layer="25">20K</text>
@@
 <attribute name="SPICEPREFIX" value="R" x="-10.16" y="24.5364" size="1.778" layer="27" rot="R180" display="off"/>
 </element>
-<element name="U2" library="myOwnLib" package="MY_IC_SO16" value="CH552G" x="17.78" y="5.9944" smashed="yes">
+<element name="U2" library="myOwnLib" package="MY_IC_SO16" value="CH549G" x="17.78" y="5.9944" smashed="yes">
 <attribute name="LCSC" value="C111292" x="45.72" y="2.1844" size="1.778" layer="27" display="off"/>
 <attribute name="VALUE" x="13.716" y="5.3594" size="1.27" layer="27" ratio="10"/>
@@
 <attribute name="SPICEPREFIX" value="R" x="26.67" y="1.4224" size="1.778" layer="27" rot="R180" display="off"/>
 </element>
-<element name="LED2" library="BeagleBone_Black_Wireless" library_urn="urn:adsk.eagle:library:6644236" package="GHI-BASICCOMPONENTS_0805-LED" package3d_urn="urn:adsk.eagle:package:6644356/2" value="P3.3" x="26.67" y="3.7084" smashed="yes" rot="R90"/>
+<element name="LED2" library="BeagleBone_Black_Wireless" library_urn="urn:adsk.eagle:library:6644236" package="GHI-BASICCOMPONENTS_0805-LED" package3d_urn="urn:adsk.eagle:package:6644356/2" value="P2.2" x="26.67" y="3.7084" smashed="yes" rot="R90"/>
 <element name="GOLD_ORB_SM1" library="oshw" package="OSHW_8MM" value="OSHWLOGOLOGO8MM" x="30.0736" y="7.366" smashed="yes" rot="MR0"/>
 <element name="J4" library="SparkFun-Connectors" library_urn="urn:adsk.eagle:library:513" package="USB-A-SMT-MALE" package3d_urn="urn:adsk.eagle:package:38305/1" value="USB_A_SMT_MALE" x="-5.334" y="5.9944" smashed="yes">
@@
 <wire x1="5.6524" y1="6.985" x2="5.616" y2="7.0214" width="0.254" layer="1"/>
 </signal>
-<signal name="P1.1">
+<signal name="P3.4">
 <contactref element="U2" pad="9"/>
 <contactref element="J1" pad="2"/>
@@
 <wire x1="20.2438" y1="1.0922" x2="20.5232" y2="1.0922" width="0.2032" layer="1"/>
 </signal>
-<signal name="P3.4">
+<signal name="P2.4">
 <contactref element="U2" pad="11"/>
 <contactref element="J2" pad="7"/>
@@
 <wire x1="23.3969125" y1="6.90643125" x2="22.8310875" y2="6.90643125" width="0.2032" layer="1"/>
 </signal>
-<signal name="P3.3">
+<signal name="P2.2">
 <contactref element="U2" pad="10"/>
 <contactref element="J2" pad="6"/>
@@
 <wire x1="29.718" y1="3.9116" x2="28.702" y2="2.8956" width="0.2032" layer="1"/>
 </signal>
-<signal name="P3.2">
+<signal name="P1.1">
 <contactref element="U2" pad="1"/>
 <contactref element="J2" pad="5"/>
@@
 <wire x1="22.55756875" y1="6.50003125" x2="23.209309375" y2="6.50003125" width="0.2032" layer="1"/>
 </signal>
-<signal name="P3.1">
+<signal name="P3.0">
 <contactref element="U2" pad="7"/>
 <contactref element="J2" pad="4"/>
@@
 <wire x1="22.0987125" y1="6.35" x2="18.6697125" y2="6.35" width="0.2032" layer="1"/>
 </signal>
-<signal name="P3.0">
+<signal name="P3.1">
 <contactref element="U2" pad="8"/>
 <contactref element="J2" pad="3"/>
