File: pcb/ch549Board/simpleCH549_typeC.brd (EAGLE design)
At the start: 35.6 x 12 mm, 14 parts, among them J4 USB_A_SMT_MALE, U2 CH549G

Commit message: adjust pins
Connections:
- net P1.1: now also J1.2; no longer J2.5
- net P3.0: now also J2.3; no longer J2.4
- net P3.1: now also J2.4; no longer J2.3
- net P3.4: now also J2.5; no longer J1.2
Routing:
- net P1.1: track 21.5 -> 4.10 mm, vias 3 -> 0
- net P3.4: track 17.2 -> 8.07 mm
- net +5V: track 66.7 -> 63.1 mm
- net P3.0: track 17.0 -> 18.3 mm
- net USB_D+: track 26.3 -> 27.1 mm
- net GND: track 58.6 -> 57.9 mm
- net P3.1: track 17.5 -> 16.8 mm
Other:
- board text added: "AIN1 CAP2 T2EX P1.1"
- board text added: "P3.4 T0"
- board text removed: "P1.1 T2EX CAP2 AIN1"
- board text removed: "T0 P3.4"

Commit message: update board
Parts:
- removed F1: (no value), adafruit:R1206
- added C3: 0.1uF, rcl:C0805K
- added J3: 629722000214, Wurth_Connectors_WR-USB:629722000214
- added U1: MCP1703CB, linear:SOT23
- J4: value USB_A_SMT_MALE -> (none); device SparkFun-Connectors:USB-A-SMT-MALE -> SparkFun-Connectors:1X02_NO_SILK
- moved J4 15.5 mm to (10.2, 5.99), turned to 270 degrees
- moved C1 4.71 mm to (15.2, 6.50)
- moved C2 4.70 mm to (15.2, 8.79)
- moved J1 4.70 mm to (12.7, 0.91)
- moved J2 4.70 mm to (12.7, 11.1)
- moved GOLD_ORB_SM1 4.70 mm to (34.8, 7.37)
- moved LED1 4.70 mm to (31.4, 8.28)
- moved LED2 4.70 mm to (31.4, 3.71)
- moved R1 4.70 mm to (31.4, 5.99)
- moved R2 4.70 mm to (31.4, 10.6)
- moved R3 4.70 mm to (31.4, 1.42)
- moved S1 4.70 mm to (36.8, 5.99)
- moved U2 4.70 mm to (22.5, 5.99)
Connections:
- new net VUSB: C3.1, J3.A4, J3.A9, J3.B4, J3.B9, J4.2, U1.3
- net +5V: now also U1.2; no longer F1.1, F1.2, J4.VBUS1
- net GND: now also C3.2, J3.A1, J3.A12, J3.B1, J3.B12, J4.1, U1.1; no longer J4.GND1
- net P1.4: now also J3.A5
- net P1.5: now also J3.B5
- net USB_D+: now also J3.A6, J3.B6; no longer J4.D+1
- net USB_D-: now also J3.A7, J3.B7; no longer J4.D-1
Routing:
- net GND: track 57.9 -> 97.6 mm, vias 4 -> 5
- net VUSB: track 0.00 -> 32.7 mm, vias 0 -> 1
- net P1.4: track 2.89 -> 30.5 mm, vias 0 -> 2
- net P1.5: track 2.37 -> 22.5 mm, vias 0 -> 2
- net USB_D+: track 27.1 -> 35.7 mm, vias 3 -> 5
- net USB_D-: track 16.4 -> 25.0 mm
- net +5V: track 63.1 -> 54.8 mm
- net RST: track 9.31 -> 10.1 mm
Other:
- board size 35.6 x 12 mm -> 40.6 x 12 mm

Commit message: board finish
Parts:
- added J5: (no value), SparkFun-Connectors:1X02_NO_SILK
- moved LED2 6.46 mm to (34.2, 9.53), turned to 0 degrees
- moved R1 2.25 mm to (33.4, 5.08), turned to 270 degrees
- moved LED1 1.59 mm to (30.4, 9.53), turned to 0 degrees
- moved R3 1.53 mm to (32.9, 1.50), turned to 0 degrees
- moved R2 1.39 mm to (32.3, 9.53), turned to 90 degrees
- moved GOLD_ORB_SM1 1.27 mm to (36.0, 7.37)
- moved S1 1.27 mm to (38.1, 5.99)
Connections:
- net GND: now also J5.1
- net VUSB: now also J5.2
Routing:
- net GND: track 97.6 -> 115.3 mm, vias 5 -> 4
- net N$2: track 2.33 -> 11.7 mm, vias 0 -> 2
- net P1.5: track 22.5 -> 28.5 mm
- net N$1: track 19.1 -> 13.4 mm, vias 2 -> 1
- net VUSB: track 32.7 -> 37.5 mm
- net P2.2: track 21.2 -> 18.5 mm
- net USB_D+: track 35.7 -> 35.2 mm
- net +5V: track 54.8 -> 54.6 mm, vias 3 -> 5
Other:
- board size 40.6 x 12 mm -> 41.9 x 12 mm
- board text added: "+"
- board text added: "-"
- board text added: "CH549 STICK PD"
- board text removed: "CH552 STICK"
- board text removed: "D+"
- board text removed: "D-"
- board text removed: "F"
