File: pcb/powerDeliveryBoard/CH552_typeC_Power_Delivery.sch (EAGLE design)
At the start: 14 parts, among them J4 USB_A_SMT_MALE, U2 CH552G

Commit message: make some progress
Parts:
- removed F1: (no value), adafruit:PTCFUSE-1206
- added C3, C4: 0.1uF, rcl:C-EUC0805K
- added D1, D2, D3, D4, D5, D6, D7, D8: (no value), diode:DIODE-SOD123
- added J3: 629722000214, Wurth_Connectors_WR-USB:629722000214
- added J5: (no value), SparkFun-Connectors:CONN_021X02_NO_SILK
- added R4: 14.7K, rcl:R-US_R0805
- added R5: 2K, rcl:R-US_R0805
- added R6, R7: 1K, rcl:R-US_R0805
- added U1: MCP1703CB, linear:MCP1703CB
- J4: value USB_A_SMT_MALE -> (none); device SparkFun-Connectors:USB_A_SMT_MALE -> SparkFun-Connectors:CONN_021X02_NO_SILK
Connections:
- new net N$4: D2.C, D3.A
- new net N$5: D3.C, D4.A
- new net N$6: D5.C, D7.A
- new net N$7: D7.C, D8.A
- new net VUSB: C3.1, J3.VBUS, J3.VBUS1, J3.VBUS2, J3.VBUS3, J4.2, J5.2, U1.VI
- net +5V: now also C4.1, R4.1, U1.VO; no longer F1.1, F1.2, J4.VBUS
- net GND: now also C3.2, C4.2, J3.GND, J3.GND1, J3.GND2, J3.GND3, J4.1, J5.1, R5.2, U1.GND; no longer J4.GND
- net P1.4: now also D1.A, D2.A, J3.CC1, R6.2
- net P1.5: now also D5.A, D6.A, J3.CC2, R7.2
- net P1.6: now also D1.C, R6.1
- net P1.7: now also D6.C, R7.1
- net P3.2: now also R4.2, R5.1
- net P3.4: now also D4.C, D8.C
- net USB_D+: now also J3.D+1, J3.D+2; no longer J4.D+
- net USB_D-: now also J3.D-1, J3.D-2; no longer J4.D-
Other:
- note added: "3 diodes to clamp voltage to 1V in PD trasmitting (regular+schottky+schottky) resistor to limit driving current schottky diode to improve low level driving"
- note added: "Any res combo to get 0.6V for BMC decode"
